File: driver/attiny1l.brd (EAGLE design)
At the start: 160 x 100 mm, 7 parts, among them IC1 ATTiny85, IC2 74AHC1G00DCK, IC3 74AHC1G00DCK, IC4 LB1973MMFP10S, J1 AVR_SPI_PRG_6NS

Commit message: trying to find got placement
Parts:
- moved IC2 4.49 mm to (45.1, 55.2), turned to 90 degrees
Connections:
- net N$10 renamed OUT1
- net N$11 renamed OUT2
- net N$8 renamed OUT4
- net N$9 renamed OUT3
Routing:
- net OUT2: track 0.00 -> 5.24 mm
- net OUT4: track 0.00 -> 4.78 mm
- net OUT1: track 0.00 -> 4.60 mm
- net OUT3: track 0.00 -> 4.43 mm
- removed copper zone on layer 1, net GND
Changed lines of the file:
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@@
 <layer number="14" name="Route14" color="1" fill="6" visible="no" active="no"/>
 <layer number="15" name="Route15" color="4" fill="6" visible="no" active="no"/>
-<layer number="16" name="Bottom" color="1" fill="1" visible="yes" active="yes"/>
+<layer number="16" name="Bottom" color="1" fill="1" visible="no" active="no"/>
 <layer number="17" name="Pads" color="2" fill="1" visible="yes" active="yes"/>
 <layer number="18" name="Vias" color="2" fill="1" visible="yes" active="yes"/>
@@
 necessary adjustments and save your customized
 design rules under a new name.</description>
-<param name="layerSetup" value="(1*16)"/>
+<param name="layerSetup" value="1"/>
 <param name="mtCopper" value="0.035mm 0.035mm 0.035mm 0.035mm 0.035mm 0.035mm 0.035mm 0.035mm 0.035mm 0.035mm 0.035mm 0.035mm 0.035mm 0.035mm 0.035mm 0.035mm"/>
 <param name="mtIsolate" value="1.5mm 0.15mm 0.2mm 0.15mm 0.2mm 0.15mm 0.2mm 0.15mm 0.2mm 0.15mm 0.2mm 0.15mm 0.2mm 0.15mm 0.2mm"/>
@@
 <param name="mdDrill" value="8mil"/>
 <param name="mdSmdStop" value="0mil"/>
-<param name="msWidth" value="10mil"/>
+<param name="msWidth" value="6mil"/>
 <param name="msDrill" value="24mil"/>
 <param name="msMicroVia" value="9.99mm"/>
@@
 <autorouter>
 <pass name="Default">
-<param name="RoutingGrid" value="50mil"/>
+<param name="RoutingGrid" value="5mil"/>
 <param name="tpViaShape" value="round"/>
 <param name="PrefDir.1" value="|"/>
@@
 <param name="PrefDir.14" value="0"/>
 <param name="PrefDir.15" value="0"/>
-<param name="PrefDir.16" value="-"/>
+<param name="PrefDir.16" value="0"/>
 <param name="cfVia" value="8"/>
 <param name="cfNonPref" value="5"/>
@@
 <attribute name="OC_FARNELL" value="9171568" x="25.4" y="67.31" size="1.778" layer="27" rot="R90" display="off"/>
 </element>
-<element name="IC2" library="74xx-little-de" package="SC70-5" value="74AHC1G00DCK" x="41.91" y="52.07" rot="R270"/>
+<element name="IC2" library="74xx-little-de" package="SC70-5" value="74AHC1G00DCK" x="45.085" y="55.245" rot="R90"/>
 <element name="IC3" library="74xx-little-de" package="SC70-5" value="74AHC1G00DCK" x="45.085" y="46.99" rot="R90"/>
 <element name="IC4" library="LB1937M" package="SSOP10" value="LB1973MMFP10S" x="46.99" y="50.8"/>
@@
 <contactref element="IC2" pad="4"/>
 <contactref element="IC4" pad="2"/>
-<wire x1="42.76" y1="51.42" x2="43.79" y2="51.8" width="0" layer="19" extent="1-1"/>
+<wire x1="43.79" y1="51.8" x2="44.235" y2="55.895" width="0" layer="19" extent="1-1"/>
 </signal>
 <signal name="IN1">
@@
 <contactref element="IC2" pad="1"/>
 <contactref element="IC1" pad="3"/>
-<wire x1="41.06" y1="52.07" x2="43.79" y2="50.8" width="0" layer="19" extent="1-1"/>
-<wire x1="41.06" y1="52.72" x2="41.06" y2="52.07" width="0" layer="19" extent="1-1"/>
-<wire x1="23.724" y1="50.155" x2="41.06" y2="52.07" width="0" layer="19" extent="1-1"/>
+<wire x1="45.935" y1="55.245" x2="45.935" y2="54.595" width="0" layer="19" extent="1-1"/>
+<wire x1="43.79" y1="50.8" x2="45.935" y2="55.245" width="0" layer="19" extent="1-1"/>
+<wire x1="23.724" y1="50.155" x2="43.79" y2="50.8" width="0" layer="19" extent="1-1"/>
 </signal>
 <signal name="GND">
@@
 <contactref element="J1" pad="6"/>
 <contactref element="SV2" pad="4"/>
-<polygon width="0.4064" layer="1" isolate="0.4064">
-<vertex x="1.27" y="66.675"/>
-<vertex x="1.27" y="37.465"/>
-<vertex x="63.5" y="37.465"/>
-<vertex x="63.5" y="67.31"/>
-<vertex x="1.27" y="67.31"/>
-</polygon>
+<wire x1="45.935" y1="47.64" x2="45.935" y2="55.895" width="0" layer="19" extent="1-1"/>
+<wire x1="50.19" y1="48.8" x2="45.935" y2="47.64" width="0" layer="19" extent="1-1"/>
+<wire x1="23.724" y1="51.425" x2="45.935" y2="55.895" width="0" layer="19" extent="1-1"/>
+<wire x1="22.86" y1="45.085" x2="23.724" y2="51.425" width="0" layer="19" extent="1-1"/>
+<wire x1="5.08" y1="53.34" x2="23.724" y2="51.425" width="0" layer="19" extent="1-1"/>
 </signal>
 <signal name="+5V">
@@
 <contactref element="J1" pad="2"/>
 <contactref element="SV2" pad="1"/>
-<wire x1="42.76" y1="52.72" x2="43.79" y2="52.8" width="0" layer="19" extent="1-1"/>
+<wire x1="43.79" y1="52.8" x2="44.235" y2="54.595" width="0" layer="19" extent="1-1"/>
 <wire x1="44.235" y1="46.34" x2="43.79" y2="52.8" width="0" layer="19" extent="1-1"/>
-<wire x1="17.78" y1="45.085" x2="42.76" y2="52.72" width="0" layer="19" extent="1-1"/>
+<wire x1="17.78" y1="45.085" x2="44.235" y2="46.34" width="0" layer="19" extent="1-1"/>
 <wire x1="16.916" y1="47.625" x2="17.78" y2="45.085" width="0" layer="19" extent="1-1"/>
 <wire x1="5.08" y1="45.72" x2="16.916" y2="47.625" width="0" layer="19" extent="1-1"/>
@@
 <wire x1="5.08" y1="48.26" x2="16.916" y2="48.895" width="0" layer="19" extent="1-1"/>
 </signal>
-<signal name="N$8">
+<signal name="OUT4">
 <contactref element="IC4" pad="10"/>
 <contactref element="SV1" pad="1"/>
-<wire x1="50.19" y1="52.8" x2="54.61" y2="54.61" width="0" layer="19" extent="1-1"/>
-</signal>
-<signal name="N$9">
+<wire x1="50.19" y1="52.8" x2="54.61" y2="54.61" width="0.2032" layer="1"/>
+</signal>
+<signal name="OUT3">
 <contactref element="IC4" pad="9"/>
 <contactref element="SV1" pad="2"/>
-<wire x1="50.19" y1="51.8" x2="54.61" y2="52.07" width="0" layer="19" extent="1-1"/>
-</signal>
-<signal name="N$10">
+<wire x1="50.19" y1="51.8" x2="54.61" y2="52.07" width="0.2032" layer="1"/>
+</signal>
+<signal name="OUT1">
 <contactref element="IC4" pad="8"/>
 <contactref element="SV1" pad="3"/>
-<wire x1="50.19" y1="50.8" x2="54.61" y2="49.53" width="0" layer="19" extent="1-1"/>
-</signal>
-<signal name="N$11">
+<wire x1="50.19" y1="50.8" x2="54.61" y2="49.53" width="0.2032" layer="1"/>
+</signal>
+<signal name="OUT2">
 <contactref element="IC4" pad="7"/>
 <contactref element="SV1" pad="4"/>
-<wire x1="50.19" y1="49.8" x2="54.61" y2="46.99" width="0" layer="19" extent="1-1"/>
+<wire x1="50.19" y1="49.8" x2="54.61" y2="46.99" width="0.2032" layer="1"/>
 </signal>
 </signals>
