File: driver/arduino_drivershield.sch (EAGLE design)
At the start: 13 parts, among them IC1 LB1973M, IC2 LB1973M, IC3 74HC14D, U1 ARDUINO_SHIELDLABEL

Commit message: second group
Parts:
- added IC10, IC11, IC4, IC5, IC7, IC8: LB1973M, LB1973M:LB1973M
- added IC12, IC6, IC9: 74HC14D, 74xx-eu:74HC14D
Connections:
- new net N$17: IC4.OUT2, JP4.4
- new net N$18: IC4.OUT1, JP4.3
- new net N$19: IC4.OUT2@1, JP4.2
- new net N$20: IC4.OUT4, JP4.1
- new net N$21: IC5.OUT2, JP5.4
- new net N$22: IC5.OUT1, JP5.3
- new net N$23: IC5.OUT2@1, JP5.2
- new net N$24: IC5.OUT4, JP5.1
- new net N$25: IC4.IN3, IC6A.O
- new net N$26: IC4.IN2, IC6B.O
- new net N$33: IC4.IN1, IC6B.I, U1.D7
- new net N$34: IC4.IN4, IC6A.I, U1.*D6
- new net N$35: IC5.IN4, IC6E.I, U1.D8
- new net N$36: IC5.IN1, IC6F.I, U1.*D9
- new net N$37: IC5.IN3, IC6E.O
- new net N$38: IC5.IN2, IC6F.O
- new net N$39: IC7.OUT2, JP6.4
- new net N$40: IC7.OUT1, JP6.3
- new net N$41: IC7.OUT2@1, JP6.2
- new net N$42: IC7.OUT4, JP6.1
- new net N$43: IC8.OUT2, JP7.4
- new net N$44: IC8.OUT1, JP7.3
- new net N$45: IC8.OUT2@1, JP7.2
- new net N$46: IC8.OUT4, JP7.1
- new net N$47: IC7.IN3, IC9A.O
- new net N$48: IC7.IN2, IC9B.O
- new net N$49: IC7.IN1, IC9B.I
- new net N$50: IC7.IN4, IC9A.I
- new net N$51: IC8.IN4, IC9E.I
- new net N$52: IC8.IN1, IC9F.I
- new net N$53: IC8.IN3, IC9E.O
- new net N$54: IC8.IN2, IC9F.O
- new net N$55: IC10.OUT2, JP8.4
- new net N$56: IC10.OUT1, JP8.3
- new net N$57: IC10.OUT2@1, JP8.2
- new net N$58: IC10.OUT4, JP8.1
- new net N$59: IC11.OUT2, JP9.4
- new net N$60: IC11.OUT1, JP9.3
- new net N$61: IC11.OUT2@1, JP9.2
- new net N$62: IC11.OUT4, JP9.1
- new net N$63: IC10.IN3, IC12A.O
- new net N$64: IC10.IN2, IC12B.O
- new net N$65: IC10.IN1, IC12B.I
- new net N$66: IC10.IN4, IC12A.I
- new net N$67: IC11.IN4, IC12E.I
- new net N$68: IC11.IN1, IC12F.I
- new net N$69: IC11.IN3, IC12E.O
- new net N$70: IC11.IN2, IC12F.O
- net 5V: now also IC1.VCC, IC10.VCC, IC11.VCC, IC2.VCC, IC4.VCC, IC5.VCC, IC7.VCC, IC8.VCC
- net GND: now also IC10.GND, IC11.GND, IC4.GND, IC5.GND, IC7.GND, IC8.GND
Other:
- moved on the sheet: JP4, JP5, JP6, JP7, JP8, JP9
