File: driver/attiny1l.sch (EAGLE design)
At the start: 7 parts, among them IC1 ATTiny85, IC2 74AHC1G00DCK, IC3 74AHC1G00DCK, IC4 LB1973M, J1 AVR_SPI_PRG_6NS

Commit message: use dual NOT and added bypass caps
Parts:
- removed IC3: 74AHC1G00DCK, 74xx-little-de:74AHC1G00DCK
- added C1, C2: (no value), rcl:C-EUC0805
- IC2: value 74AHC1G00DCK -> (none); device 74xx-little-de:74AHC1G00DCK -> dp_devices:IC_BUFF_SN74LVC2G17DBV
Connections:
- removed net IN3: IC1.PB4/PCINT4/ADC2, IC2A.I0, IC2A.I1, IC4.IN3
- removed net IN4: IC2A.O, IC4.IN4
- new net N$1: IC1.PB4/PCINT4/ADC2, IC2.1A, IC4.IN3
- new net N$2: IC2.1Y, IC4.IN4
- net +5V: now also C1.1, C2.1, IC2.VCC; no longer IC2P.VCC, IC3P.VCC
- net GND: now also C1.2, C2.2, IC2.GND; no longer IC2P.GND, IC3P.GND
- net IN1/MISO: now also IC2.2A; no longer IC3A.I0, IC3A.I1
- net IN2: now also IC2.2Y; no longer IC3A.O
Changed lines of the file:
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@@
 <layer number="106" name="bPlate" color="7" fill="1" visible="no" active="yes"/>
 <layer number="107" name="Crop" color="7" fill="1" visible="no" active="yes"/>
+<layer number="108" name="centerline" color="7" fill="1" visible="yes" active="yes"/>
 <layer number="116" name="Patch_BOT" color="9" fill="4" visible="no" active="yes"/>
 <layer number="121" name="_tsilk" color="7" fill="1" visible="no" active="yes"/>
 <layer number="122" name="_bsilk" color="7" fill="1" visible="no" active="yes"/>
 <layer number="125" name="_tNames" color="7" fill="1" visible="no" active="yes"/>
+<layer number="131" name="prix" color="7" fill="1" visible="yes" active="yes"/>
+<layer number="132" name="test" color="7" fill="1" visible="yes" active="yes"/>
 <layer number="144" name="Drill_legend" color="7" fill="1" visible="no" active="yes"/>
 <layer number="151" name="HeatSink" color="7" fill="1" visible="no" active="yes"/>
@@
 <parts>
 <part name="IC1" library="atmel" deviceset="TINY13" device="SU" technology="-20" value="ATTiny85"/>
-<part name="IC2" library="74xx-little-de" deviceset="74*1G00" device="DCK" technology="AHC"/>
-<part name="IC3" library="74xx-little-de" deviceset="74*1G00" device="DCK" technology="AHC"/>
-<part name="GND1" library="supply1" deviceset="GND" device=""/>
-<part name="GND2" library="supply1" deviceset="GND" device=""/>
 <part name="GND3" library="supply1" deviceset="GND" device=""/>
 <part name="GND4" library="supply1" deviceset="GND" device=""/>
 <part name="P+1" library="supply1" deviceset="+5V" device=""/>
-<part name="P+2" library="supply1" deviceset="+5V" device=""/>
-<part name="P+3" library="supply1" deviceset="+5V" device=""/>
 <part name="P+4" library="supply1" deviceset="+5V" device=""/>
 <part name="J1" library="SparkFun-Connectors" deviceset="AVR_SPI_PRG_6" device="NS"/>
@@
 <part name="GND6" library="supply1" deviceset="GND" device=""/>
 <part name="IC4" library="LB1973M" deviceset="LB1973M" device=""/>
+<part name="IC2" library="dp_devices" deviceset="IC_BUFF_SN74LVC2G17" device="DBV"/>
+<part name="GND1" library="supply1" deviceset="GND" device=""/>
+<part name="P+2" library="supply1" deviceset="+5V" device=""/>
+<part name="C1" library="rcl" deviceset="C-EU" device="C0805"/>
+<part name="C2" library="rcl" deviceset="C-EU" device="C0805"/>
 </parts>
 <sheets>
@@
 <instances>
 <instance part="IC1" gate="G$1" x="30.48" y="78.74" rot="R180"/>
-<instance part="IC2" gate="A" x="104.14" y="81.28"/>
-<instance part="IC3" gate="A" x="104.14" y="63.5"/>
-<instance part="IC3" gate="P" x="104.14" y="50.8" rot="R270"/>
-<instance part="IC2" gate="P" x="104.14" y="91.44" rot="R270"/>
-<instance part="GND1" gate="1" x="96.52" y="48.26"/>
-<instance part="GND2" gate="1" x="96.52" y="88.9"/>
 <instance part="GND3" gate="1" x="50.8" y="86.36" rot="R180"/>
 <instance part="GND4" gate="1" x="180.34" y="71.12"/>
 <instance part="P+1" gate="1" x="119.38" y="86.36"/>
-<instance part="P+2" gate="1" x="111.76" y="93.98"/>
-<instance part="P+3" gate="1" x="111.76" y="53.34"/>
 <instance part="P+4" gate="1" x="50.8" y="63.5" rot="R180"/>
 <instance part="J1" gate="G$1" x="66.04" y="106.68"/>
@@
 <instance part="GND6" gate="1" x="33.02" y="55.88" rot="R180"/>
 <instance part="IC4" gate="G$1" x="149.86" y="78.74"/>
+<instance part="IC2" gate="G$1" x="93.98" y="53.34"/>
+<instance part="GND1" gate="1" x="83.82" y="55.88" rot="R270"/>
+<instance part="P+2" gate="1" x="114.3" y="55.88" rot="R270"/>
+<instance part="C1" gate="G$1" x="38.1" y="96.52" rot="R90"/>
+<instance part="C2" gate="G$1" x="121.92" y="93.98" rot="R90"/>
 </instances>
 <busses>
@@
 <net name="IN2" class="0">
 <segment>
-<pinref part="IC3" gate="A" pin="O"/>
-<wire x1="111.76" y1="63.5" x2="119.38" y2="63.5" width="0.1524" layer="91"/>
-<wire x1="119.38" y1="63.5" x2="119.38" y2="73.66" width="0.1524" layer="91"/>
 <pinref part="IC4" gate="G$1" pin="IN2"/>
-</segment>
-</net>
-<net name="IN4" class="0">
-<segment>
-<pinref part="IC2" gate="A" pin="O"/>
-<wire x1="111.76" y1="81.28" x2="119.38" y2="81.28" width="0.1524" layer="91"/>
-<pinref part="IC4" gate="G$1" pin="IN4"/>
+<pinref part="IC2" gate="G$1" pin="2Y"/>
+<wire x1="111.76" y1="50.8" x2="119.38" y2="50.8" width="0.1524" layer="91"/>
+<wire x1="119.38" y1="50.8" x2="119.38" y2="73.66" width="0.1524" layer="91"/>
 </segment>
 </net>
 <net name="IN1/MISO" class="0">
 <segment>
-<pinref part="IC3" gate="A" pin="I0"/>
-<pinref part="IC3" gate="A" pin="I1"/>
-<wire x1="99.06" y1="66.04" x2="99.06" y2="60.96" width="0.1524" layer="91"/>
-<wire x1="99.06" y1="66.04" x2="99.06" y2="71.12" width="0.1524" layer="91"/>
-<wire x1="99.06" y1="71.12" x2="114.3" y2="71.12" width="0.1524" layer="91"/>
 <wire x1="114.3" y1="71.12" x2="114.3" y2="76.2" width="0.1524" layer="91"/>
 <wire x1="114.3" y1="76.2" x2="119.38" y2="76.2" width="0.1524" layer="91"/>
-<junction x="99.06" y="66.04"/>
-<junction x="99.06" y="60.96"/>
 <pinref part="IC1" gate="G$1" pin="PB1/PCINT1/AIN1/OC0B/INT0/MISO"/>
 <wire x1="50.8" y1="71.12" x2="53.34" y2="71.12" width="0.1524" layer="91"/>
-<junction x="99.06" y="71.12"/>
 <pinref part="J1" gate="G$1" pin="1"/>
-<wire x1="53.34" y1="71.12" x2="99.06" y2="71.12" width="0.1524" layer="91"/>
+<wire x1="53.34" y1="71.12" x2="71.12" y2="71.12" width="0.1524" layer="91"/>
+<wire x1="71.12" y1="71.12" x2="114.3" y2="71.12" width="0.1524" layer="91"/>
 <wire x1="58.42" y1="109.22" x2="53.34" y2="109.22" width="0.1524" layer="91"/>
 <wire x1="53.34" y1="109.22" x2="53.34" y2="71.12" width="0.1524" layer="91"/>
 <junction x="53.34" y="71.12"/>
 <pinref part="IC4" gate="G$1" pin="IN1"/>
-</segment>
-</net>
-<net name="IN3" class="0">
-<segment>
-<wire x1="119.38" y1="78.74" x2="111.76" y2="78.74" width="0.1524" layer="91"/>
-<wire x1="111.76" y1="78.74" x2="111.76" y2="73.66" width="0.1524" layer="91"/>
-<pinref part="IC2" gate="A" pin="I1"/>
-<wire x1="111.76" y1="73.66" x2="99.06" y2="73.66" width="0.1524" layer="91"/>
-<wire x1="99.06" y1="73.66" x2="99.06" y2="78.74" width="0.1524" layer="91"/>
-<pinref part="IC2" gate="A" pin="I0"/>
-<wire x1="99.06" y1="78.74" x2="99.06" y2="83.82" width="0.1524" layer="91"/>
-<junction x="99.06" y="78.74"/>
-<junction x="99.06" y="83.82"/>
-<pinref part="IC1" gate="G$1" pin="PB4/PCINT4/ADC2"/>
-<wire x1="50.8" y1="78.74" x2="99.06" y2="78.74" width="0.1524" layer="91"/>
-<pinref part="IC4" gate="G$1" pin="IN3"/>
+<pinref part="IC2" gate="G$1" pin="2A"/>
+<wire x1="86.36" y1="50.8" x2="71.12" y2="50.8" width="0.1524" layer="91"/>
+<wire x1="71.12" y1="50.8" x2="71.12" y2="71.12" width="0.1524" layer="91"/>
+<junction x="71.12" y="71.12"/>
 </segment>
 </net>
 <net name="GND" class="0">
-<segment>
-<pinref part="IC3" gate="P" pin="GND"/>
-<pinref part="GND1" gate="1" pin="GND"/>
-</segment>
-<segment>
-<pinref part="IC2" gate="P" pin="GND"/>
-<pinref part="GND2" gate="1" pin="GND"/>
-</segment>
 <segment>
 <pinref part="IC1" gate="G$1" pin="GND"/>
 <pinref part="GND3" gate="1" pin="GND"/>
+<wire x1="50.8" y1="83.82" x2="63.5" y2="83.82" width="0.1524" layer="91"/>
+<wire x1="63.5" y1="83.82" x2="63.5" y2="96.52" width="0.1524" layer="91"/>
+<pinref part="C1" gate="G$1" pin="2"/>
+<wire x1="63.5" y1="96.52" x2="43.18" y2="96.52" width="0.1524" layer="91"/>
 </segment>
 <segment>
@@
 <pinref part="GND4" gate="1" pin="GND"/>
 <pinref part="IC4" gate="G$1" pin="GND"/>
+<wire x1="180.34" y1="73.66" x2="185.42" y2="73.66" width="0.1524" layer="91"/>
+<wire x1="185.42" y1="73.66" x2="185.42" y2="60.96" width="0.1524" layer="91"/>
+<wire x1="185.42" y1="60.96" x2="134.62" y2="60.96" width="0.1524" layer="91"/>
+<wire x1="134.62" y1="60.96" x2="134.62" y2="93.98" width="0.1524" layer="91"/>
+<pinref part="C2" gate="G$1" pin="2"/>
+<wire x1="134.62" y1="93.98" x2="127" y2="93.98" width="0.1524" layer="91"/>
+</segment>
+<segment>
+<pinref part="IC2" gate="G$1" pin="GND"/>
+<pinref part="GND1" gate="1" pin="GND"/>
 </segment>
 </net>
 <net name="+5V" class="0">
-<segment>
-<pinref part="IC2" gate="P" pin="VCC"/>
-<pinref part="P+2" gate="1" pin="+5V"/>
-</segment>
-<segment>
-<pinref part="IC3" gate="P" pin="VCC"/>
-<pinref part="P+3" gate="1" pin="+5V"/>
-</segment>
 <segment>
 <pinref part="IC1" gate="G$1" pin="VCC"/>
 <pinref part="P+4" gate="1" pin="+5V"/>
+<wire x1="50.8" y1="66.04" x2="66.04" y2="66.04" width="0.1524" layer="91"/>
+<wire x1="66.04" y1="66.04" x2="66.04" y2="91.44" width="0.1524" layer="91"/>
+<pinref part="C1" gate="G$1" pin="1"/>
+<wire x1="66.04" y1="91.44" x2="35.56" y2="91.44" width="0.1524" layer="91"/>
+<wire x1="35.56" y1="91.44" x2="35.56" y2="96.52" width="0.1524" layer="91"/>
 </segment>
 <segment>
@@
 <pinref part="P+1" gate="1" pin="+5V"/>
 <pinref part="IC4" gate="G$1" pin="VCC"/>
+<wire x1="119.38" y1="83.82" x2="114.3" y2="83.82" width="0.1524" layer="91"/>
+<wire x1="114.3" y1="83.82" x2="114.3" y2="93.98" width="0.1524" layer="91"/>
+<pinref part="C2" gate="G$1" pin="1"/>
+<wire x1="114.3" y1="93.98" x2="119.38" y2="93.98" width="0.1524" layer="91"/>
+</segment>
+<segment>
+<pinref part="IC2" gate="G$1" pin="VCC"/>
+<pinref part="P+2" gate="1" pin="+5V"/>
 </segment>
 </net>
@@
 </segment>
 </net>
+<net name="N$1" class="0">
+<segment>
+<pinref part="IC1" gate="G$1" pin="PB4/PCINT4/ADC2"/>
+<pinref part="IC2" gate="G$1" pin="1A"/>
+<wire x1="50.8" y1="78.74" x2="86.36" y2="78.74" width="0.1524" layer="91"/>
+<wire x1="86.36" y1="78.74" x2="86.36" y2="60.96" width="0.1524" layer="91"/>
+<pinref part="IC4" gate="G$1" pin="IN3"/>
+<wire x1="86.36" y1="78.74" x2="119.38" y2="78.74" width="0.1524" layer="91"/>
+<junction x="86.36" y="78.74"/>
+</segment>
+</net>
+<net name="N$2" class="0">
+<segment>
+<pinref part="IC2" gate="G$1" pin="1Y"/>
+<wire x1="111.76" y1="60.96" x2="111.76" y2="81.28" width="0.1524" layer="91"/>
+<pinref part="IC4" gate="G$1" pin="IN4"/>
+<wire x1="111.76" y1="81.28" x2="119.38" y2="81.28" width="0.1524" layer="91"/>
+</segment>
+</net>

Commit message: added a debugging led
Parts:
- added LED1: (no value), SparkFun-LED:LED0603
Connections:
- new net N$3: IC1.PB3/PCINT3/CLKI/ADC3, LED1.A
- net GND: now also LED1.C
Changed lines of the file:
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@@
 <part name="C1" library="rcl" deviceset="C-EU" device="C0805"/>
 <part name="C2" library="rcl" deviceset="C-EU" device="C0805"/>
+<part name="LED1" library="SparkFun-LED" deviceset="LED" device="0603"/>
 </parts>
 <sheets>
@@
 <instance part="C1" gate="G$1" x="38.1" y="96.52" rot="R90"/>
 <instance part="C2" gate="G$1" x="121.92" y="93.98" rot="R90"/>
+<instance part="LED1" gate="G$1" x="68.58" y="96.52" rot="R270"/>
 </instances>
 <busses>
@@
 <pinref part="C1" gate="G$1" pin="2"/>
 <wire x1="63.5" y1="96.52" x2="43.18" y2="96.52" width="0.1524" layer="91"/>
+<pinref part="LED1" gate="G$1" pin="C"/>
+<junction x="63.5" y="96.52"/>
 </segment>
 <segment>
@@
 </segment>
 </net>
+<net name="N$3" class="0">
+<segment>
+<pinref part="IC1" gate="G$1" pin="PB3/PCINT3/CLKI/ADC3"/>
+<pinref part="LED1" gate="G$1" pin="A"/>
+<wire x1="50.8" y1="76.2" x2="71.12" y2="76.2" width="0.1524" layer="91"/>
+<wire x1="71.12" y1="76.2" x2="71.12" y2="96.52" width="0.1524" layer="91"/>
+</segment>
+</net>

Commit message: otoh this way I can sample our input voltage when not driving the led...
Connections:
- net +5V: now also LED1.A
- net GND: no longer LED1.C
- net N$3: now also LED1.C; no longer LED1.A
Other:
- moved on the sheet: LED1
Changed lines of the file:
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@@
 <instance part="C1" gate="G$1" x="38.1" y="96.52" rot="R90"/>
 <instance part="C2" gate="G$1" x="121.92" y="93.98" rot="R90"/>
-<instance part="LED1" gate="G$1" x="68.58" y="96.52" rot="R270"/>
+<instance part="LED1" gate="G$1" x="63.5" y="76.2" rot="R270"/>
 </instances>
 <busses>
@@
 <wire x1="63.5" y1="83.82" x2="63.5" y2="96.52" width="0.1524" layer="91"/>
 <pinref part="C1" gate="G$1" pin="2"/>
-<wire x1="63.5" y1="96.52" x2="43.18" y2="96.52" width="0.1524" layer="91"/>
-<pinref part="LED1" gate="G$1" pin="C"/>
-<junction x="63.5" y="96.52"/>
+<wire x1="43.18" y1="96.52" x2="63.5" y2="96.52" width="0.1524" layer="91"/>
 </segment>
 <segment>
@@
 <pinref part="P+4" gate="1" pin="+5V"/>
 <wire x1="50.8" y1="66.04" x2="66.04" y2="66.04" width="0.1524" layer="91"/>
-<wire x1="66.04" y1="66.04" x2="66.04" y2="91.44" width="0.1524" layer="91"/>
+<wire x1="66.04" y1="66.04" x2="66.04" y2="76.2" width="0.1524" layer="91"/>
 <pinref part="C1" gate="G$1" pin="1"/>
+<wire x1="66.04" y1="76.2" x2="66.04" y2="91.44" width="0.1524" layer="91"/>
 <wire x1="66.04" y1="91.44" x2="35.56" y2="91.44" width="0.1524" layer="91"/>
 <wire x1="35.56" y1="91.44" x2="35.56" y2="96.52" width="0.1524" layer="91"/>
+<pinref part="LED1" gate="G$1" pin="A"/>
+<junction x="66.04" y="76.2"/>
 </segment>
 <segment>
@@
 <net name="N$3" class="0">
 <segment>
+<pinref part="LED1" gate="G$1" pin="C"/>
 <pinref part="IC1" gate="G$1" pin="PB3/PCINT3/CLKI/ADC3"/>
-<pinref part="LED1" gate="G$1" pin="A"/>
-<wire x1="50.8" y1="76.2" x2="71.12" y2="76.2" width="0.1524" layer="91"/>
-<wire x1="71.12" y1="76.2" x2="71.12" y2="96.52" width="0.1524" layer="91"/>
+<wire x1="58.42" y1="76.2" x2="50.8" y2="76.2" width="0.1524" layer="91"/>
 </segment>
 </net>
