File: driver/attiny_driver.brd (EAGLE design)
At the start: 160 x 100 mm, 10 parts, among them IC1 ATTiny85, IC4 LB1973M, J1 AVR_SPI_PRG_6NS

Commit message: DRC loaded
Parts:
- JP1: device pinhead:1X02 -> pinhead:1X04
- moved LED1 8.47 mm to (24.8, 50.2), turned to 180 degrees
- moved C1 7.75 mm to (24.8, 52.1), flipped to the bottom, turned to 90 degrees
- moved JP1 7.62 mm to (31.8, 52.1)
- moved J1 1.42 mm to (20.3, 51.4)
- moved IC1 0.90 mm to (28.6, 46.4), flipped to the bottom, turned to 270 degrees
Connections:
- net GND: now also JP1.4; no longer JP1.2
- net SCL/SCK: now also JP1.2
- net SDA/MOSI: now also JP1.3
Routing:
- added copper zone on layer 1, net GND
- added copper zone on layer 16, net GND
Other:
- board text added: "GND SCL SDA 5V"
