File: driver/attiny_driver.sch (EAGLE design)
At the start: 10 parts, among them IC1 ATTiny85, IC4 LB1973M, J1 AVR_SPI_PRG_6NS

Commit message: DRC loaded
Parts:
- JP1: device pinhead:PINHD-1X2 -> pinhead:PINHD-1X4
Connections:
- net GND: now also JP1.4; no longer JP1.2
- net SCL/SCK: now also JP1.2
- net SDA/MOSI: now also JP1.3
Changed lines of the file:
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@@
 <part name="C2" library="rcl" deviceset="C-EU" device="C0805"/>
 <part name="LED1" library="SparkFun-LED" deviceset="LED" device="0603"/>
-<part name="JP1" library="pinhead" deviceset="PINHD-1X2" device=""/>
 <part name="JP2" library="pinhead" deviceset="PINHD-1X2" device=""/>
 <part name="JP3" library="pinhead" deviceset="PINHD-1X2" device=""/>
+<part name="JP1" library="pinhead" deviceset="PINHD-1X4" device=""/>
 </parts>
 <sheets>
@@
 <instance part="C2" gate="G$1" x="121.92" y="93.98" rot="R90"/>
 <instance part="LED1" gate="G$1" x="63.5" y="76.2" rot="R270"/>
-<instance part="JP1" gate="G$1" x="35.56" y="40.64" rot="R270"/>
 <instance part="JP2" gate="G$1" x="187.96" y="81.28"/>
 <instance part="JP3" gate="G$1" x="187.96" y="76.2"/>
+<instance part="JP1" gate="A" x="35.56" y="50.8" rot="R270"/>
 </instances>
 <busses>
@@
 </segment>
 <segment>
-<pinref part="JP1" gate="G$1" pin="2"/>
 <pinref part="GND6" gate="1" pin="GND"/>
-<wire x1="35.56" y1="43.18" x2="33.02" y2="43.18" width="0.1524" layer="91"/>
-<wire x1="33.02" y1="43.18" x2="33.02" y2="53.34" width="0.1524" layer="91"/>
+<pinref part="JP1" gate="A" pin="4"/>
 </segment>
 </net>
@@
 </segment>
 <segment>
-<pinref part="JP1" gate="G$1" pin="1"/>
 <pinref part="P+6" gate="1" pin="+5V"/>
-<wire x1="38.1" y1="43.18" x2="40.64" y2="43.18" width="0.1524" layer="91"/>
-<wire x1="40.64" y1="43.18" x2="40.64" y2="53.34" width="0.1524" layer="91"/>
+<pinref part="JP1" gate="A" pin="1"/>
 </segment>
 </net>
@@
 <wire x1="60.96" y1="60.96" x2="35.56" y2="60.96" width="0.1524" layer="91"/>
 <wire x1="35.56" y1="60.96" x2="35.56" y2="53.34" width="0.1524" layer="91"/>
+<pinref part="JP1" gate="A" pin="3"/>
 </segment>
 </net>
@@
 <junction x="55.88" y="73.66"/>
 <wire x1="38.1" y1="53.34" x2="38.1" y2="58.42" width="0.1524" layer="91"/>
+<pinref part="JP1" gate="A" pin="2"/>
 </segment>
 </net>
